File: electronics/electromagneticMarbleMachine.kicad_sch (KiCad schematic)
At the start: 102 parts, among them K1 SPST Relay, Q1 2N2222, Q10 PT334-6B, Q11 2N2222, Q12 2N2222, Q2 2N2222, Q3 PT334-6B, Q4 PT334-6B, Q5 2N2222, Q6 2N2222, Q7 2N2222, Q8 PT334-6B, Q9 PT334-6B, SW1 Latching Pushbotton, SW2 Cherry MX Switch, SW3 DPST Switch, SW4 Cherry MX Switch, SW5 SPST Switch, U1 LM2576T-5, U2 LM2576T-12, U3 ATmega328P-PU, U4 LM2576T-5, U5 UGN3503UA, Y1 20MHz

Commit message: idk
idk
Parts:
- removed D1, D31, D4: 6A10 Diode, Diode_THT:D_A-405_P10.16mm_Horizontal, symbol Diode:1N4007
- removed D3: Red LED, LED_THT:LED_D5.0mm, symbol dk_LED-Indication-Discrete:151033RS03000
- removed R2: 330Ω, symbol Device:R
- removed SW3: DPST Switch, symbol Switch:SW_DPST
- added D2, D31, D4: 1N5408, Diode_THT:D_DO-201AD_P15.24mm_Horizontal, symbol Diode:1N5408
- added SW2: spdt microswitch, Button_Switch_THT:SW_Slide-03_Wuerth-WS-SLTV_10x2.5x6.4_P2.54mm, symbol Switch:SW_Wuerth_450301014042
- C10, C11, C12, C13, C9: value 680uF -> 1000uF; footprint (none) -> custom:ALF70G102EH450
- D10, D12, D22, D24, D26, D30: value 70TPS12 -> CLA50E1200HB; footprint (none) -> LIB_CLA50E1200HB:TO546P530X1586X2594-3P
- D11, D13, D14, D21, D23, D25, D27, D28, D29, D32: value 6A10 Diode -> 6A10; footprint Diode_THT:D_A-405_P10.16mm_Horizontal -> LIB_6A10:DIOAD4425W130L885D885
- D15, D16, D17, D6, D7: footprint LED_THT:LED_D5.0mm -> LIB_QED234:QED234
- D3: renamed from D2; value 6A10 Diode -> 6A10; footprint Diode_THT:D_A-405_P10.16mm_Horizontal -> LIB_6A10:DIOAD4425W130L885D885
- D9: value 6A10 Diode -> 6A10
- K1: value SPST Relay -> 5V relay module
- Q1, Q11, Q12, Q2, Q5, Q6, Q7: footprint Package_TO_SOT_THT:TO-92_Inline -> LIB_P2N2222A:P2N2222A
- Q10, Q3, Q4, Q8, Q9: footprint (none) -> LIB_PT334-6B:PT3346B
- R10: renamed from R11; footprint (none) -> Resistor_THT:R_Axial_DIN0207_L6.3mm_D2.5mm_P10.16mm_Horizontal
- R14: renamed from R15; footprint (none) -> Resistor_THT:R_Axial_DIN0207_L6.3mm_D2.5mm_P10.16mm_Horizontal
- R16: renamed from R17; footprint (none) -> Resistor_THT:R_Axial_DIN0207_L6.3mm_D2.5mm_P10.16mm_Horizontal
- R2: renamed from R3; footprint (none) -> Resistor_THT:R_Axial_DIN0207_L6.3mm_D2.5mm_P10.16mm_Horizontal
- R3: renamed from R4; footprint (none) -> Resistor_THT:R_Axial_DIN0207_L6.3mm_D2.5mm_P10.16mm_Horizontal
- R4: renamed from R5; footprint (none) -> Resistor_THT:R_Axial_DIN0207_L6.3mm_D2.5mm_P10.16mm_Horizontal
- R5: renamed from R6; footprint (none) -> Resistor_THT:R_Axial_DIN0207_L6.3mm_D2.5mm_P10.16mm_Horizontal
- R7: renamed from R8; footprint (none) -> Resistor_THT:R_Axial_DIN0207_L6.3mm_D2.5mm_P10.16mm_Horizontal
- R8: renamed from R9; footprint (none) -> Resistor_THT:R_Axial_DIN0207_L6.3mm_D2.5mm_P10.16mm_Horizontal
- R9: renamed from R10; footprint (none) -> Resistor_THT:R_Axial_DIN0207_L6.3mm_D2.5mm_P10.16mm_Horizontal
- SW3: renamed from SW2; footprint Cherry MX:Cherry-MX_PCB-Mounted -> PCM_Switch_Keyboard_Cherry_MX:SW_Cherry_MX_PCB
- SW4: footprint Cherry MX:Cherry-MX_PCB-Mounted -> PCM_Switch_Keyboard_Cherry_MX:SW_Cherry_MX_PCB
- U1, U4: footprint Package_TO_SOT_THT:TO-220-5_Vertical -> LIB_LM2576T-5.0_NOPB:LM2576T50NOPB
- U2: footprint Package_TO_SOT_THT:TO-220-5_Vertical -> LIB_LM2576T-12_NOPB:TO170P483X1016X1611-5P
- U5: footprint (none) -> LIB_UGN3503UA:UGN3503UA
- V1: value 20V 3.25A -> 65W Vin
- V3: footprint (none) -> custom:9V Battery Holder
- renumbered R12 to R11, R13 to R12, R14 to R13, R16 to R15, R7 to R6
Connections:
- net 12V: no longer Q1.1 (C), Q10.1 (C), Q2.1 (C), Q4.1 (C), Q5.1 (C), Q6.1 (C), Q7.1 (C), Q8.1 (C), Q9.1 (C), R10.1, R5.1, R8.1, R9.1
- net 20V: now also SW2.1 (B)
- net 5Va: now also Q1.1 (C), Q10.1 (C), Q2.1 (C), Q4.1 (C), Q5.1 (C), Q6.1 (C), Q7.1 (C), Q8.1 (C), Q9.1 (C), R10.1, R5.1, R8.1, R9.1
- net Earth: now also D2.1 (K), D31.1 (K), D4.1 (K)
- net at L1.1, U1.4 (VO): now also D2.2 (A)
- net at L8.1, U4.2 (VO): now also D31.2 (A)
- net at D3.2 (A): now also SW2.3 (A)
- net at L2.1, U2.4 (VO): now also D4.2 (A)
Other:
- moved on the sheet: D3, L3, L4, L5, L6, L7

Commit message: final PCB added
a bunch of simulation and KiCad files.
Parts:
- removed C14: 0.1uF, Capacitor_THT:C_Disc_D4.3mm_W1.9mm_P5.00mm, symbol Device:C_Small
- removed C3: 100uF, Capacitor_THT:C_Radial_D8.0mm_H11.5mm_P3.50mm, symbol Device:C_Polarized_Small
- removed C4: 470uF, Capacitor_THT:C_Radial_D8.0mm_H11.5mm_P3.50mm, symbol Device:C_Polarized_Small
- removed D10, D12, D22, D24, D26, D30: CLA50E1200HB, LIB_CLA50E1200HB:TO546P530X1586X2594-3P, symbol customSymbols:70TPS12PBF
- removed D15, D16, D17, D6: IR LED, LIB_QED234:QED234, symbol dk_LED-Indication-Discrete:151033RS03000
- removed D18: White LED, LED_THT:LED_D5.0mm, symbol dk_LED-Indication-Discrete:151033RS03000
- removed D2, D31: 1N5408, Diode_THT:D_DO-201AD_P15.24mm_Horizontal, symbol Diode:1N5408
- removed D21, D23, D25, D27, D28, D3: 6A10, LIB_6A10:DIOAD4425W130L885D885, symbol Diode:1N4007
- removed D9: 6A10, Diode_THT:D_A-405_P10.16mm_Horizontal, symbol Diode:1N4007
- removed DS1: ~, symbol customSymbols:voltmeter_display
- removed L7: 100uH, symbol Device:L
- removed SW1: Latching Pushbotton, symbol customSymbols:latching_pushbutton
- removed SW4: Cherry MX Switch, PCM_Switch_Keyboard_Cherry_MX:SW_Cherry_MX_PCB, symbol Cherry_MX:Cherry_MX
- removed U2: LM2576T-12, LIB_LM2576T-12_NOPB:TO170P483X1016X1611-5P, symbol Regulator_Switching:LM2576T-5
- added BZ1: buzzer, custom:Buzzer, symbol Device:Buzzer
- added C1, C2: 0.01uF, Capacitor_THT:C_Disc_D4.3mm_W1.9mm_P5.00mm, symbol Device:C_Small
- added D1, D43: 1N5822, Diode_THT:D_DO-201AD_P15.24mm_Horizontal, symbol Diode:1N5822
- added D10, D25, D26, D27, D28, D9: 1N5408, Diode_THT:D_DO-201AD_P15.24mm_Horizontal, symbol Diode:1N5408
- added D12, D16, D17, D2, D30, D31, D32, D33, D35, D36, D38, D39: 6A10, LIB_6A10:DIOAD4425W130L885D885, symbol Diode:1N4007
- added D15, D18, D34, D37, D40, D41: CLA50E1200HB, LIB_CLA50E1200HB:TO546P530X1586X2594-3P, symbol custom:CLA50E1200HB
- added D21: IR LED, LIB_QED234:QED234, symbol dk_LED-Indication-Discrete:151033RS03000
- added D22, D23, D24, D42, D7: 5mm LED, LED_THT:LED_D5.0mm, symbol dk_LED-Indication-Discrete:151033RS03000
- added D3: White LED, LED_THT:LED_D5.0mm, symbol dk_LED-Indication-Discrete:151033RS03000
- added J1: SSD1306, custom:128x64OLED, symbol Connector:Conn_01x04_Socket
- added J10, J11, J12, J15, J2, J8, J9: ~, custom:1x1 2.54mm header, symbol Connector_Generic_MountingPin:Conn_01x01_MountingPin
- added J16: Conn_01x03_MountingPin, custom:1x3 2.54mm header, symbol Connector_Generic_MountingPin:Conn_01x03_MountingPin
- added J3, J5: Shunt, Connector_PinHeader_2.54mm:PinHeader_1x02_P2.54mm_Vertical, symbol Connector_Generic_MountingPin:Conn_01x02_MountingPin
- added J4: Conn_01x03_MountingPin, custom:1x2 2.54mm header, symbol Connector_Generic_MountingPin:Conn_01x03_MountingPin
- added J6, J7: Conn_01x14_MountingPin, custom:1x14 2.54mm header, symbol Connector_Generic_MountingPin:Conn_01x14_MountingPin
- added R15, R31, R32, R33, R36: 2k2Ω, Resistor_THT:R_Axial_DIN0207_L6.3mm_D2.5mm_P10.16mm_Horizontal, symbol Device:R
- added R17, R28, R29, R30: 10kΩ, Resistor_THT:R_Axial_DIN0207_L6.3mm_D2.5mm_P10.16mm_Horizontal, symbol Device:R
- added R18, R19: 270Ω, Resistor_THT:R_Axial_DIN0207_L6.3mm_D2.5mm_P10.16mm_Horizontal, symbol Device:R
- added R20, R21, R22: 390Ω, Resistor_THT:R_Axial_DIN0207_L6.3mm_D2.5mm_P10.16mm_Horizontal, symbol Device:R
- added R23, R24, R25: 1k2Ω, Resistor_THT:R_Axial_DIN0207_L6.3mm_D2.5mm_P10.16mm_Horizontal, symbol Device:R
- added R26: 900Ω, Resistor_THT:R_Axial_DIN0207_L6.3mm_D2.5mm_P10.16mm_Horizontal, symbol Device:R
- added R27: 47Ω, Resistor_THT:R_Axial_DIN0207_L6.3mm_D2.5mm_P10.16mm_Horizontal, symbol Device:R
- added R34: 10k0Ω, Resistor_THT:R_Axial_DIN0207_L6.3mm_D2.5mm_P10.16mm_Horizontal, symbol Device:R
- added RV1: 1MΩ Pot, custom:potentiometer, symbol Device:R_Potentiometer
- added RV2: 10kΩ Pot, custom:potentiometerOFFBOARD, symbol Device:R_Potentiometer
- added SW1: Pushbutton, Button_Switch_THT:SW_PUSH_6mm, symbol Cherry_MX:Cherry_MX
- added U2: NE555P, Package_DIP:DIP-8_W7.62mm, symbol Timer:NE555P
- added U3, U5, U6, U7, U8: 4N28, Package_DIP:DIP-6_W7.62mm, symbol Isolator:4N28
- C10, C11, C12, C13, C9: footprint custom:ALF70G102EH450 -> custom:officialCAP
- C15: renamed from C16; footprint Capacitor_THT:C_Radial_D8.0mm_H11.5mm_P3.50mm -> Capacitor_THT:C_Radial_D10.0mm_H12.5mm_P5.00mm
- C4: renamed from C2; footprint Capacitor_THT:C_Radial_D8.0mm_H11.5mm_P3.50mm -> Capacitor_THT:C_Radial_D10.0mm_H12.5mm_P5.00mm
- D19, D20: value White LED -> IR LED; footprint LED_THT:LED_D5.0mm -> LIB_QED234:QED234
- D5: value Green LED -> IR LED; footprint LED_THT:LED_D5.0mm -> LIB_QED234:QED234
- D8: value White LED -> 5mm LED
- K1: value 5V relay module -> 5V relay; footprint (none) -> custom:5v relay
- L1: footprint (none) -> custom:Inductor
- L2: value 150uH -> 100uH; footprint (none) -> custom:Coil Socket
- L3, L4, L5, L6: footprint (none) -> custom:Coil Socket
- L7: renamed from L8; footprint (none) -> custom:Inductor
- L8: renamed from L9; value 12V solenoid -> Solenoid; footprint (none) -> custom:solenoid_WIRED
- Q12: value 2N2222 -> BC639
- R10: value 330Ω -> 270Ω
- R11, R6: value 330Ω -> 390Ω
- R12, R13, R2: value 330Ω -> 10kΩ
- R14: value 10kΩ -> 2k2Ω
- R16: value 1KΩ -> 270Ω
- R3: value 330Ω -> 910kΩ
- R35: renamed from R15; value 200W 1kΩ -> 200W 1k0Ω; footprint (none) -> custom:200W Resistor
- R4: value 1KΩ -> 2k2Ω
- R5: value 330Ω -> 2k0Ω
- R7: value 1KΩ -> 390Ω
- R8, R9: value 330Ω -> 1k2Ω
- SW2: value spdt microswitch -> SPDT Microswitch; footprint Button_Switch_THT:SW_Slide-03_Wuerth-WS-SLTV_10x2.5x6.4_P2.54mm -> custom:microswitch
- SW3: value Cherry MX Switch -> N/C Pushbutton; footprint PCM_Switch_Keyboard_Cherry_MX:SW_Cherry_MX_PCB -> custom:button_or_keyswitch
- SW4: renamed from SW5; footprint (none) -> custom:button_or_keyswitch
- U1: footprint LIB_LM2576T-5.0_NOPB:LM2576T50NOPB -> LIB_LM2576T-12_NOPB:TO170P483X1016X1611-5P
- U9: renamed from U4; footprint LIB_LM2576T-5.0_NOPB:LM2576T50NOPB -> LIB_LM2576T-12_NOPB:TO170P483X1016X1611-5P
- V1: value 65W Vin -> 20V Vin; footprint (none) -> custom:20Vin
- V2: footprint (none) -> custom:405Vin
- renumbered C15 to C14, C1 to C3, D32 to D44, D7 to D6, U5 to U10, U3 to U4
Connections:
- net 20V: now also Q12.1 (C), D2.1 (K), J3.1 (Pin_1)
- net 405V+: now also D13.2 (A), D16.2 (A), D32.2 (A), D35.2 (A), D38.2 (A); no longer C10.1, C11.1, C12.1, C13.1, C9.1, D11.2 (A)
- net 5Va: now also D5.1, R7.2, J2.1 (Pin_1), R20.2, R21.2, R22.2, R23.1, R24.1, R25.1, R27.1, U3.5, U5.5, U6.5, U7.5, U8.5; no longer Q10.1 (C), Q4.1 (C), Q8.1 (C), Q9.1 (C), R10.1, R11.2, R12.2, R13.2, R5.1, R6.2, R8.1
- net 5Vd: now also R8.1, J1.1 (Pin_1), J15.1 (Pin_1), J16.1 (Pin_1), J6.7 (Pin_7), J7.8 (Pin_8), J7.9 (Pin_9), RV2.3, U2.4 (R), U2.8 (VCC); no longer Q3.1 (C)
- net 9V: no longer R7.1
- net Earth: now also C10.2, C11.2, C12.2, C13.2, C9.2, D19.2, D20.2, D4.2 (A), K1.4, L8.2 (-), R11.1, R12.2, R13.2, R14.1, V1.2 (-), V2.3 (VOUT-), BZ1.2 (-), D1.2 (A), D15.1, D18.1, D21.2, D34.1, D37.1, D40.1, D41.1, J10.1 (Pin_1), J11.1 (Pin_1), J12.1 (Pin_1), J4.2 (Pin_2), J8.1 (Pin_1), J9.1 (Pin_1), R15.2, R28.2, R29.2, R30.2, R31.2, R32.2, R33.2, R34.1, R36.1, RV1.1; no longer C14.2, C15.2, C5.2, C6.2, C7.2, C8.2, D4.1 (K), D5.2, K1.3, L8.-, Q11.3 (E), R3.2, SW3.1, U10.2 (GND), U4.22 (GND), U4.8 (GND), U9.3 (GND), U9.5 (~{ON}/OFF), V3.2 (-)
- net bleed: now also R26.1, U8.4; no longer R14.2, U4.15 (D9(PWM))
- net charge: now also D4.1 (K), K1.3, U5.4; no longer K1.2, U4.17 (D11(PWM))
- net discharge: now also Q1.2 (B), D7.1, U6.4; no longer R4.2, U4.16 (D10(PWM))
- net solenoid: now also Q12.2 (B), D42.1, U7.4; no longer R16.1, U4.14 (D8)
- net voltmeter: now reaches R3.1
- net voltmeter: now also C9.1, D11.2 (A), D13.1 (K), D14.1 (K), L2.1
- net at SW2.2 (C): now also J5.1 (Pin_1)
- net bypass: now reaches SW2.3 (A)
- net bypass: now also K1.1, J3.2 (Pin_2)
- net at Q11.2 (B): now also R26.2; no longer R14.1
- net safety: now reaches D11.1 (K)
- net safety: now also D29.1 (K), R35.2, D12.1 (K), D30.1 (K), D31.1 (K)
- net A2: now reaches U10.3 (VO)
- net A2: now also U4.25 (A2), J16.3 (Pin_3), J7.4 (Pin_4)
- net at R6.1: now also D3.1; no longer D6.1
- net at R2.1: now also R3.2, U2.7 (DIS); no longer D5.1
- net at D8.1: now also Q2.2 (B), Q4.1 (C), R9.2; no longer R5.2
- net at Q11.1 (C): now also R27.2; no longer R7.2
- net at R1.2, U4.1 (~{RESET}): now also J6.1 (Pin_1), SW1.2; no longer SW3.2
- net at D20.1: now also R21.1; no longer R10.2
- net at L5.1: now also C12.1, D30.2 (A), D35.1 (K), D36.1 (K)
- net at C5.1, U4.9 (OSC1), Y1.1: now also J6.9 (Pin_9)
- net Earth_Clean: now reaches R16.2
- net Earth_Clean: now also C14.2, C15.2, C5.2, C6.2, C7.2, C8.2, Q3.2 (E), R10.2, R4.2, R5.2, SW3.1, U10.2 (GND), U4.22 (GND), U4.8 (GND), U9.3 (GND), U9.5 (~{ON}/OFF), V3.2 (-), C1.1, C2.1, D3.2, D43.2 (A), J1.2 (Pin_2), J16.2 (Pin_2), J6.8 (Pin_8), J7.7 (Pin_7), R17.2, R18.2, R19.2, RV2.1, SW1.1, U2.1 (GND); no longer Q12.2 (B)
- net at L1.1, U1.4 (VO): now also D1.1 (K)
- net at L7.1, U9.2 (VO): now also D43.1 (K)
- net at Q7.2 (B): now also Q10.1 (C), D24.1, R25.2; no longer D20.2
- net at Q7.3 (E): now also D27.2 (A), R30.1
- net at R4.1: now also U3.2; no longer Q1.2 (B)
- net at D19.1: now also R20.1; no longer R9.2
- net at C6.1, U4.10 (OSC2), Y1.2: now also J6.10 (Pin_10)
- net at U4.11 (D5(PWM)): now also J6.11 (Pin_11)
- net at U4.12 (D6(PWM)): now also J6.12 (Pin_12)
- net D7: now reaches U4.13 (D7)
- net D7: now also SW3.2, J6.13 (Pin_13)
- net D12: now reaches U4.18 (D12)
- net D12: now also J7.11 (Pin_11), U7.1
- net at U4.19 (D13): now also R6.2, J7.10 (Pin_10); no longer R2.2
- net at U4.2 (D0(RX)): now also J6.2 (Pin_2)
- net A0: now reaches U4.23 (A0)
- net A0: now also J7.6 (Pin_6), R17.1, RV2.2
- net A1: now reaches U4.24 (A1)
- net A1: now also Q3.1 (C), R8.2, J7.5 (Pin_5)
- net at U4.26 (A3): now also J7.3 (Pin_3)
- net at U4.3 (D1(TX)): now also J6.3 (Pin_3)
- net at U4.4 (D2): now also J6.4 (Pin_4)
- net at U4.5 (D3(PWM)): now also J6.5 (Pin_5)
- net at U4.6 (D4): now also J6.6 (Pin_6)
- net at Q5.3 (E): now also D25.2 (A), R28.1
- net at R12.1: now also Q1.3 (E), D9.2 (A)
- net at D8.2: now also R15.1; no longer Q2.2 (B)
- net at Q2.3 (E): now also R13.1, D10.2 (A)
- net at L3.1: now also C10.1, D12.2 (A), D16.1 (K), D17.1 (K); no longer D13.1 (K)
- net at L4.1: now also C11.1, D29.2 (A), D32.1 (K), D33.1 (K); no longer D14.1 (K)
- net at Q6.2 (B): now also Q9.1 (C), D23.1, R24.2; no longer D19.2
- net at Q6.3 (E): now also D26.2 (A), R29.1
- net at L6.1: now also C13.1, D31.2 (A), D38.1 (K), D39.1 (K)
- net at D44.1 (K), Q12.3 (E): now also L8.1 (+); no longer L8.+
- net at Q5.2 (B): now also Q8.1 (C), D22.1, R23.2
- net at V2.1 (VIN+): now also K1.2; no longer K1.4
- net 12V: no longer names the net of L2.2
- net 12V: now also D14.2 (A), D15.2; no longer Q12.1 (C)
- removed net 405V-: C10.2, C11.2, C12.2, C13.2, C9.2, D13.2 (A), D14.2 (A), D29.2 (A), L3.2, L4.2, L5.2, L6.2, R35.1, V2.3 (VOUT-)
- net hallEffect renamed SCL
- net SCL: now also J1.3 (Pin_3), J7.1 (Pin_1)
- net receiverIR renamed SDA
- net SDA: now also J1.4 (Pin_4), J7.2 (Pin_2); no longer Q3.2 (E)
- new net: D17.2 (A), D18.2, L3.2
- new net: R18.1, U7.2
- new net: D10.1 (K), D18.3
- new net: D33.2 (A), D34.2, L4.2
- new net: D25.1 (K), D34.3
- new net: D42.2, R36.2
- new net: R16.1, U6.2
- new net: D41.2, R35.1
- new net: R10.1, U5.2
- new net: D15.3, D9.1 (K)
- new net: D28.2 (A), Q11.3 (E), R34.2
- new net: D36.2 (A), D37.2, L5.2
- new net: D24.2, R33.1
- new net: D6.1, R7.1
- new net: D2.2 (A), J4.1 (Pin_1), V1.1 (+)
- new net: C2.2, R2.2
- new net: J5.2 (Pin_2), RV1.3
- new net: D28.1 (K), D41.3
- new net: U2.3 (Q), U3.1
- new net: U2.2 (TR), U2.6 (THR)
- new net: C1.2, U2.5 (CV)
- new net: D39.2 (A), D40.2, L6.2
- new net: D27.1 (K), D40.3
- new net: BZ1.1 (+), RV1.2
- new net: D5.2, R11.2
- new net: R19.1, U8.2
- new net: D26.1 (K), D37.3
- new net: D21.1, R22.1
- new net: D23.2, R32.1
- new net: D22.2, R31.1
- new net: D7.2, R14.2
- new net D10: J7.13 (Pin_13), U4.16 (D10(PWM)), U6.1
- new net D11: J7.12 (Pin_12), U4.17 (D11(PWM)), U5.1
- new net D8: J6.14 (Pin_14), R5.1, U3.4, U4.14 (D8)
- new net D9: J7.14 (Pin_14), U4.15 (D9(PWM)), U8.1
- no-connect marks 0 -> 5
Other:
- note added: "biased hall effect sensor"
- note removed: "hall effect sensor"
- company: James Bray - 11EST1 -> james bray - 11EST1
- title: Marble Machine Circuitry -> electromagnetic marble machine
- moved on the sheet: C3, C4, C5, C6, C7, C8, D44, D6, K1, L1, L8, Q1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
