File: kicadFiles/electromagneticMarbleMachine.kicad_sch (KiCad schematic)
At the start: 151 parts, among them J1 SSD1306, J16 Conn_01x03_MountingPin, J3 Shunt, J4 Conn_01x03_MountingPin, J5 Shunt, J6 Conn_01x14_MountingPin, J7 Conn_01x14_MountingPin, K1 5V relay, Q1 2N2222, Q10 PT334-6B, Q11 2N2222, Q12 BC639, Q2 2N2222, Q3 PT334-6B, Q4 PT334-6B, Q5 2N2222, Q6 2N2222, Q7 2N2222, Q8 PT334-6B, Q9 PT334-6B, SW1 Pushbutton, SW2 SPDT Microswitch, SW3 N/C Pushbutton, SW4 SPST Switch, U1 LM2576T-5, U10 UGN3503UA, U2 NE555P, U3 4N28, U4 ATmega328P-PU, U5 4N28, U6 4N28, U7 4N28, U8 4N28, U9 LM2576T-5, Y1 20MHz

Commit message: assorted files
an assortment of images and plots of my electronics have been added.
Parts:
- added R37: 5k0Ω, Resistor_THT:R_Axial_DIN0207_L6.3mm_D2.5mm_P10.16mm_Horizontal, symbol Device:R
Connections:
- net 405V+: now also R37.2; no longer V2.4 (VOUT+)
- new net: R37.1, V2.4 (VOUT+)
Changed lines of the file:
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@@
 	(wire
 		(pts
+			(xy 152.4 52.07) (xy 154.94 52.07)
+		)
+		(stroke
+			(width 0)
+			(type default)
+		)
+	)
+	(wire
+		(pts
 			(xy 119.38 111.76) (xy 151.13 111.76)
 		)
@@
 	(wire
 		(pts
+			(xy 154.94 35.56) (xy 154.94 40.64)
+		)
+		(stroke
+			(width 0)
+			(type default)
+		)
+	)
+	(wire
+		(pts
 			(xy 41.91 109.22) (xy 41.91 111.76)
 		)
@@
 	(wire
 		(pts
-			(xy 153.67 52.07) (xy 152.4 52.07)
-		)
-		(stroke
-			(width 0)
-			(type default)
-		)
-	)
-	(wire
-		(pts
 			(xy 152.4 186.69) (xy 152.4 189.23)
 		)
@@
 	(wire
 		(pts
+			(xy 154.94 52.07) (xy 154.94 48.26)
+		)
+		(stroke
+			(width 0)
+			(type default)
+		)
+	)
+	(wire
+		(pts
 			(xy 137.16 173.99) (xy 139.7 173.99)
 		)
@@
 	(global_label "405V+"
 		(shape output)
-		(at 153.67 52.07 0)
+		(at 154.94 35.56 0)
 		(fields_autoplaced yes)
 		(effects
@@
 		)
 		(property "Intersheetrefs" "${INTERSHEET_REFS}"
-			(at 160.8048 52.07 0)
+			(at 162.0748 35.56 0)
 			(effects
 				(font
@@
 					(unit 1)
 				)
+			)
+		)
+	)
+	(symbol
+		(lib_id "Device:R")
+		(at 154.94 44.45 0)
+		(mirror x)
+		(unit 1)
+		(exclude_from_sim no)
+		(in_bom yes)
+		(on_board no)
+		(dnp no)
+		(property "Reference" "R37"
+			(at 156.21 43.688 0)
+			(effects
+				(font
+					(size 1.27 1.27)
+				)
+				(justify left)
+			)
+		)
+		(property "Value" "5k0Ω"
+			(at 156.21 45.466 0)
+			(effects
+				(font
+					(size 1.27 1.27)
+					(bold yes)
+				)
+				(justify left)
+			)
+		)
+		(property "Footprint" "Resistor_THT:R_Axial_DIN0207_L6.3mm_D2.5mm_P10.16mm_Horizontal"
+			(at 153.162 44.45 90)
+			(effects
+				(font
+					(size 1.27 1.27)
+				)
+				(hide yes)
+			)
+		)
+		(property "Datasheet" "~"
+			(at 154.94 44.45 0)
+			(effects
+				(font
+					(size 1.27 1.27)
+				)
+				(hide yes)
+			)
+		)
+		(property "Description" ""
+			(at 154.94 44.45 0)
+			(effects
+				(font
+					(size 1.27 1.27)
+				)
+				(hide yes)
+			)
+		)
+		(pin "1"
+		)
+		(pin "2"
+		)
+		(instances
+			(project "electromagneticMarbleMachine"
+				(path "/599574c5-ce89-47df-9d8e-ef9e12b057f6"
+					(reference "R37")
+					(unit 1)
+				)

Commit message: error fixes
Parts:
- removed R37: 5k0Ω, Resistor_THT:R_Axial_DIN0207_L6.3mm_D2.5mm_P10.16mm_Horizontal, symbol Device:R
Connections:
- net 405V+: now also V2.4 (VOUT+)
Changed lines of the file:
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@@
 	(wire
 		(pts
-			(xy 152.4 52.07) (xy 154.94 52.07)
+			(xy 152.4 52.07) (xy 153.67 52.07)
 		)
 		(stroke
@@
 	(wire
 		(pts
-			(xy 154.94 35.56) (xy 154.94 40.64)
-		)
-		(stroke
-			(width 0)
-			(type default)
-		)
-	)
-	(wire
-		(pts
 			(xy 41.91 109.22) (xy 41.91 111.76)
 		)
@@
 	(wire
 		(pts
-			(xy 154.94 52.07) (xy 154.94 48.26)
-		)
-		(stroke
-			(width 0)
-			(type default)
-		)
-	)
-	(wire
-		(pts
 			(xy 137.16 173.99) (xy 139.7 173.99)
 		)
@@
 	(global_label "405V+"
 		(shape output)
-		(at 154.94 35.56 0)
+		(at 153.67 52.07 0)
 		(fields_autoplaced yes)
 		(effects
@@
 		)
 		(property "Intersheetrefs" "${INTERSHEET_REFS}"
-			(at 162.0748 35.56 0)
+			(at 160.8048 52.07 0)
 			(effects
 				(font
@@
 					(unit 1)
 				)
-			)
-		)
-	)
-	(symbol
-		(lib_id "Device:R")
-		(at 154.94 44.45 0)
-		(mirror x)
-		(unit 1)
-		(exclude_from_sim no)
-		(in_bom yes)
-		(on_board no)
-		(dnp no)
-		(property "Reference" "R37"
-			(at 156.21 43.688 0)
-			(effects
-				(font
-					(size 1.27 1.27)
-				)
-				(justify left)
-			)
-		)
-		(property "Value" "5k0Ω"
-			(at 156.21 45.466 0)
-			(effects
-				(font
-					(size 1.27 1.27)
-					(bold yes)
-				)
-				(justify left)
-			)
-		)
-		(property "Footprint" "Resistor_THT:R_Axial_DIN0207_L6.3mm_D2.5mm_P10.16mm_Horizontal"
-			(at 153.162 44.45 90)
-			(effects
-				(font
-					(size 1.27 1.27)
-				)
-				(hide yes)
-			)
-		)
-		(property "Datasheet" "~"
-			(at 154.94 44.45 0)
-			(effects
-				(font
-					(size 1.27 1.27)
-				)
-				(hide yes)
-			)
-		)
-		(property "Description" ""
-			(at 154.94 44.45 0)
-			(effects
-				(font
-					(size 1.27 1.27)
-				)
-				(hide yes)
-			)
-		)
-		(pin "1"
-		)
-		(pin "2"
-		)
-		(instances
-			(project "electromagneticMarbleMachine"
-				(path "/599574c5-ce89-47df-9d8e-ef9e12b057f6"
-					(reference "R37")
-					(unit 1)
-				)
